File: rei_pcb.kicad_pcb (KiCad board)
At the start: 2 copper layers, 333.4 x 95.3 mm, 163 parts, among them J1 SM04B-SRSS-TB(LF)(SN), SW1 SW_Push, U1 ATmega32U4-AU, Y1 16MHz

Commit message: update pcb
Parts:
- removed U1: ATmega32U4-AU, Package_QFP:TQFP-44_10x10mm_P0.8mm
- added U2: ATmega32U4RC-MU, Package_DFN_QFN:QFN-44-1EP_7x7mm_P0.5mm_EP5.2x5.2mm, B.Cu at (50.8, 100.0)
- C1, C2, C3, C4, C5, C6, C7: footprint Capacitor_SMD:C_0805_2012Metric -> Capacitor_SMD:C_0603_1608Metric
- R1, R2, R3, R4: footprint Resistor_SMD:R_0805_2012Metric -> Resistor_SMD:R_0603_1608Metric
- moved C3 53.2 mm to (50.0, 107.3), turned to 270 degrees
- moved R4 50.7 mm to (51.6, 107.3)
- moved C7 46.1 mm to (43.4, 99.9)
- moved C5 45.5 mm to (53.5, 86.9)
- moved C2 43.8 mm to (58.7, 100.0), turned to 180 degrees
- moved Y1 41.7 mm to (52.2, 90.6)
- moved SW1 40.7 mm to (49.5, 116.3)
- moved C6 40.4 mm to (50.9, 86.9), turned to 90 degrees
- moved C4 38.8 mm to (46.0, 94.7), turned to 135 degrees
- moved F1 38.4 mm to (44.3, 89.5), turned to 90 degrees
- moved R3 38.0 mm to (47.3, 110.2)
- moved C1 33.4 mm to (55.6, 94.7), turned to 45 degrees
- moved R2 32.2 mm to (46.4, 77.4)
- moved J1 31.2 mm to (47.4, 67.0), turned to 0 degrees
- moved R1 27.9 mm to (48.4, 77.3)
Routing:
- net GND: track 141.9 -> 1.08 mm, vias 5 -> 0
- net +5V: track 77.4 -> 0.00 mm, vias 5 -> 0
- net Net-(R1-Pad1): track 44.2 -> 0.00 mm, vias 2 -> 0
- net VCC: track 42.8 -> 0.00 mm, vias 2 -> 0
- net Net-(R2-Pad1): track 42.0 -> 0.00 mm, vias 2 -> 0
- net Net-(R3-Pad2): track 16.0 -> 0.00 mm, vias 2 -> 0
- net Net-(C6-Pad1): track 11.9 -> 2.28 mm
- net ROW3: track 309.6 -> 317.9 mm
- net Net-(C5-Pad1): track 7.22 -> 0.00 mm
- net D-: track 6.64 -> 0.00 mm
- net D+: track 6.64 -> 0.00 mm
- net Net-(C4-Pad1): track 6.57 -> 0.00 mm
- net Net-(R4-Pad1): track 6.21 -> 0.00 mm
Other:
- net class Default: clearance 0.2 -> 0.1778; via_dia 0.8 -> 0.6
- net class Power: clearance 0.2 -> 0.1778; trace_width 0.381 -> 0.254; via_dia 0.8 -> 0.6
- rule trace_clearance: 0.2 -> 0.1778

Commit message: PCB initial complete
Parts:
- moved SW1 30.7 mm to (36.6, 88.5), turned to 180 degrees
- moved R3 22.5 mm to (41.5, 88.5), turned to 270 degrees
- moved C1 7.95 mm to (48.0, 92.7), turned to 135 degrees
- moved R2 1.84 mm to (48.3, 77.2)
- moved R1 1.84 mm to (46.6, 77.2)
- moved F1 1.31 mm to (45.5, 89.0)
- moved C4 0.97 mm to (45.2, 95.2)
- moved C3 0.64 mm to (50.0, 108.0), turned to 90 degrees
- moved R4 0.64 mm to (51.6, 108.0)
Connections:
- J1 pad 1: GND -> VCC
- J1 pad 2: D+ -> D-
- J1 pad 3: D- -> D+
- J1 pad 4: VCC -> GND
- U2 pad 10: Net-(U2-Pad10) -> ROW2
- U2 pad 11: Net-(U2-Pad11) -> ROW1
- U2 pad 18: Net-(U2-Pad18) -> ROW0
- U2 pad 19: Net-(U2-Pad19) -> COL4
- U2 pad 20: Net-(U2-Pad20) -> COL3
- U2 pad 21: Net-(U2-Pad21) -> COL2
- U2 pad 22: Net-(U2-Pad22) -> COL1
- U2 pad 24: Net-(U2-Pad24) -> +5V
- U2 pad 25: Net-(U2-Pad25) -> COL5
- U2 pad 26: Net-(U2-Pad26) -> COL6
- U2 pad 27: Net-(U2-Pad27) -> COL7
- U2 pad 28: Net-(U2-Pad28) -> COL8
- U2 pad 29: Net-(U2-Pad29) -> COL9
- U2 pad 30: Net-(U2-Pad30) -> COL10
- U2 pad 31: Net-(U2-Pad31) -> COL11
- U2 pad 32: Net-(U2-Pad32) -> COL12
- U2 pad 36: Net-(U2-Pad36) -> COL14
- U2 pad 37: Net-(U2-Pad37) -> COL13
- U2 pad 38: Net-(U2-Pad38) -> COL15
- U2 pad 39: Net-(U2-Pad39) -> COL0
- U2 pad 40: Net-(U2-Pad40) -> ROW4
- U2 pad 41: Net-(U2-Pad41) -> ROW3
- U2 pad 44: Net-(U2-Pad24) -> +5V
Routing:
- net COL14: track 44.0 -> 410.4 mm, vias 0 -> 1
- net COL15: track 92.4 -> 408.4 mm
- net COL13: track 82.9 -> 385.2 mm, vias 0 -> 1
- net COL11: track 67.0 -> 330.2 mm, vias 0 -> 1
- net COL12: track 110.4 -> 357.3 mm, vias 0 -> 1
- net COL10: track 96.6 -> 305.1 mm, vias 0 -> 1
- net COL9: track 67.0 -> 259.7 mm, vias 0 -> 1
- net COL8: track 67.0 -> 234.2 mm, vias 0 -> 1
- net COL7: track 88.0 -> 227.0 mm, vias 0 -> 1
- net COL6: track 67.0 -> 194.1 mm, vias 0 -> 1
- net GND: track 1.08 -> 112.5 mm
- net COL5: track 67.0 -> 174.3 mm, vias 0 -> 1
- net COL4: track 67.0 -> 145.0 mm, vias 0 -> 1
- net ROW0: track 308.2 -> 380.4 mm, vias 0 -> 2
- net +5V: track 0.00 -> 66.7 mm, vias 0 -> 7
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- added copper zone on B.Cu, net GND
- added copper zone on F.Cu, net GND
Other:
- outline, holes or cut-outs redrawn

Commit message: Gerber files
Routing:
- removed copper zone on F.Cu, net GND
Changed lines of the file:
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@@
     (visible_elements 7FFFFFFF)
     (pcbplotparams
-      (layerselection 0x010fc_ffffffff)
-      (usegerberextensions false)
+      (layerselection 0x010f0_ffffffff)
+      (usegerberextensions true)
       (usegerberattributes false)
       (usegerberadvancedattributes false)
@@
       (outputformat 1)
       (mirror false)
-      (drillshape 1)
+      (drillshape 0)
       (scaleselection 1)
-      (outputdirectory ""))
+      (outputdirectory "Gerbers/"))
   )
   (net 0 "")
@@
       )
     )
-  )
-  (zone (net 1) (net_name GND) (layer F.Cu) (hatch edge 0.508)
-    (connect_pads (clearance 0.508))
-    (min_thickness 0.254)
-    (fill yes (arc_segments 32) (thermal_gap 0.508) (thermal_bridge_width 0.508))
-    (polygon
-      (pts
-        (xy 49.53 84.836) (xy 49.403 84.836) (xy 49.403 84.709) (xy 49.53 84.709)
-      )
-    )

Commit message: Completed PCB
Parts:
- added LOGO: Val**, Downloads:LOGO (10), F.Cu at (209.7, 112.0)
- added LOGO: Val**, Downloads:LOGO (9), F.Cu at (152.8, 111.1)
- MX3, MX6, MX73, MX76: footprint MX_Only:MXOnly-2U-FLIPPED -> MX_Only:MXOnly-2U-NoLED
- MX65: footprint MX_Only:MXOnly-2.25U-FLIPPED-ReversedStabilizers -> MX_Only:MXOnly-2.25U-ReversedStabilizers-NoLED
- moved F1 1.65 mm to (45.5, 87.4)
- moved D16 1.41 mm to (113.0, 61.1)
- moved D10 1.14 mm to (70.2, 118.5)
- moved D49 1.14 mm to (279.8, 118.5)
- moved D58 1.14 mm to (327.6, 118.5)
- moved D35 1.06 mm to (203.5, 99.1)
- moved D19 1.02 mm to (117.9, 118.5)
- moved D36 1.02 mm to (198.8, 118.5)
- moved D41 0.95 mm to (217.8, 42.0)
- moved D61 0.94 mm to (320.4, 80.0)
- moved D22 0.93 mm to (136.8, 80.0)
- moved D37 0.92 mm to (198.7, 42.0)
- moved D59 0.92 mm to (293.9, 42.0)
- moved D20 0.92 mm to (122.5, 42.0)
- moved D55 0.91 mm to (284.4, 61.1)
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Routing:
- net ROW1: track 346.4 -> 337.4 mm
- net ROW0: track 380.4 -> 371.6 mm
- net ROW3: track 325.5 -> 317.4 mm
- net ROW2: track 374.3 -> 368.6 mm
- net ROW4: track 321.4 -> 316.9 mm
- net COL13: track 385.2 -> 382.0 mm
- net COL14: track 410.4 -> 407.3 mm
- net COL11: track 330.2 -> 327.2 mm
- net COL15: track 408.4 -> 406.4 mm
- net VCC: track 16.8 -> 15.2 mm
- net Net-(D16-Pad2): track 7.29 -> 8.65 mm
- net COL4: track 145.0 -> 143.7 mm
- net Net-(D34-Pad2): track 7.09 -> 8.33 mm
- net Net-(D9-Pad2): track 7.53 -> 8.67 mm
- net Net-(D58-Pad2): track 7.75 -> 8.89 mm
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Other:
- outline, holes or cut-outs redrawn
- net class Power: trace_width 0.254 -> 0.381
