File: rei_pcb.kicad_pcb (KiCad board)
At the start: 2 copper layers, 333.4 x 95.3 mm, 163 parts, among them J1 SM04B-SRSS-TB(LF)(SN), SW1 SW_Push, U2 ATmega32U4RC-MU, Y1 16MHz

Commit message: Push update
Parts:
- removed the D51 at (265.4, 61.1)
- removed MX1, MX14, MX15, MX16, MX17, MX18, MX19, MX2, MX20, MX21, MX23, MX24, MX25, MX26, MX27, MX28, MX29, MX30, MX31, MX32, MX33, MX34, MX35, MX36, MX37, MX38, MX4, MX40, MX41, MX42, MX43, MX44, MX45, MX46, MX47, MX48, MX49, MX5, MX50, MX51, MX53, MX54, MX55, MX56, MX57, MX58, MX59, MX63, MX64, MX66, MX67, MX7, MX70, MX71, MX72, MX74, MX75, MX77, MX8: MX-NoLED, MX_Only:MXOnly-1U-NoLED
- removed MX10, MX60: MX-NoLED, MX_Only:MXOnly-1.75U-NoLED
- removed MX11: MX-NoLED, MX_Only:MXOnly-1.25U-NoLED
- removed MX12, MX61: MX-NoLED, MX_Only:MXOnly-2.25U-NoLED
- removed MX13, MX22, MX52, MX62, MX69, MX9: MX-NoLED, MX_Only:MXOnly-1.5U-NoLED
- removed MX3, MX6, MX68, MX73, MX76: MX-NoLED, MX_Only:MXOnly-2U-NoLED
- removed MX39: MX-NoLED, MX_Only:MXOnly-7U-ReversedStabilizers-NoLED
- removed MX65: MX-NoLED, MX_Only:MXOnly-2.25U-ReversedStabilizers-NoLED
- removed SW1: SW_Push, random-keyboard-parts:SKQG-1155865
- added D51 (x6): D_Small, Diode_SMD:D_SOD-123, B.Cu at (255.6, 41.3)
- added D71: D_Small, Diode_SMD:D_SOD-123, B.Cu at (339.7, 103.2)
- added D72: D_Small, Diode_SMD:D_SOD-123, B.Cu at (339.7, 112.7)
- added J2: AVR-ISP-6, random-keyboard-parts:Reset_Pretty-Mask, B.Cu at (50.0, 116.2)
- added JP1: SolderJumper_3_Open, Jumper:SolderJumper-3_P1.3mm_Open_RoundedPad1.0x1.5mm_NumberLabels, B.Cu at (347.7, 49.5)
- added JP2: SolderJumper_3_Open, Jumper:SolderJumper-3_P1.3mm_Open_RoundedPad1.0x1.5mm_NumberLabels, B.Cu at (33.3, 50.0)
- added JP3: SolderJumper_3_Open, Jumper:SolderJumper-3_P1.3mm_Open_RoundedPad1.0x1.5mm_NumberLabels, B.Cu at (62.0, 87.5)
- added MX_'1: MX-LED, MX_Only:MXOnly-1U, F.Cu at (281.0, 79.4)
- added MX_,1: MX-LED, MX_Only:MXOnly-1U, F.Cu at (233.4, 98.4)
- added MX_-1: MX-LED, MX_Only:MXOnly-1U, F.Cu at (266.7, 41.3)
- added MX_.1: MX-LED, MX_Only:MXOnly-1U, F.Cu at (252.4, 98.4)
- added MX_/1: MX-LED, MX_Only:MXOnly-1U, F.Cu at (271.5, 98.4)
- added MX_0: MX-LED, MX_Only:MXOnly-1U, F.Cu at (247.7, 41.3)
- added MX_1: MX-LED, MX_Only:MXOnly-1U, F.Cu at (76.2, 41.3)
- added MX_2: MX-LED, MX_Only:MXOnly-1U, F.Cu at (95.2, 41.3)
- added MX_3: MX-LED, MX_Only:MXOnly-1U, F.Cu at (114.3, 41.3)
- added MX_4: MX-LED, MX_Only:MXOnly-1U, F.Cu at (133.3, 41.3)
- added MX_5: MX-LED, MX_Only:MXOnly-1U, F.Cu at (152.4, 41.3)
- added MX_6: MX-LED, MX_Only:MXOnly-1U, F.Cu at (171.4, 41.3)
- added MX_7: MX-LED, MX_Only:MXOnly-1U, F.Cu at (190.5, 41.3)
- added MX_8: MX-LED, MX_Only:MXOnly-1U, F.Cu at (209.6, 41.3)
- added MX_9: MX-LED, MX_Only:MXOnly-1U, F.Cu at (228.6, 41.3)
- added MX_;1: MX-LED, MX_Only:MXOnly-1U, F.Cu at (261.9, 79.4)
- added MX_=1: MX-LED, MX_Only:MXOnly-1U, F.Cu at (285.8, 41.3)
- added MX_A1: MX-LED, MX_Only:MXOnly-1U, F.Cu at (90.5, 79.4)
- added MX_B1: MX-LED, MX_Only:MXOnly-1U, F.Cu at (176.2, 98.4)
- added MX_BSPACE1: MX-LED, MX_Only:MXOnly-2U, F.Cu at (314.3, 41.3)
- added MX_BSPACE2: MX-LED, MX_Only:MXOnly-1U, F.Cu at (304.8, 41.3)
- added MX_BSPACE3: MX-LED, MX_Only:MXOnly-1U, F.Cu at (323.9, 41.3)
- added MX_C1: MX-LED, MX_Only:MXOnly-1U, F.Cu at (138.1, 98.4)
- added MX_CLOCK1: MX-LED, MX_Only:MXOnly-1.75U, F.Cu at (64.3, 79.4)
- added MX_CLOCKSTEP1: MX-LED, MX_Only:MXOnly-1.25U-FLIPPED, F.Cu at (59.5, 79.4)
- added MX_D1: MX-LED, MX_Only:MXOnly-1U, F.Cu at (128.6, 79.4)
- added MX_E1: MX-LED, MX_Only:MXOnly-1U, F.Cu at (123.8, 60.3)
- added MX_ENTER1: MX-LED, MX_Only:MXOnly-2.25U-ReversedStabilizers, F.Cu at (311.9, 79.4)
- added MX_ESC1: MX-LED, MX_Only:MXOnly-1U, F.Cu at (33.3, 41.3)
- added MX_F1: MX-LED, MX_Only:MXOnly-1U, F.Cu at (33.3, 60.3)
- added MX_F10: MX-LED, MX_Only:MXOnly-1U, F.Cu at (147.6, 79.4)
- added MX_F1V1: MX-LED, MX_Only:MXOnly-2U, F.Cu at (33.3, 69.8)
- added MX_F2: MX-LED, MX_Only:MXOnly-1U, F.Cu at (33.3, 79.4)
- added MX_F3: MX-LED, MX_Only:MXOnly-1U, F.Cu at (33.3, 98.4)
- added MX_F3V1: MX-LED, MX_Only:MXOnly-2U, F.Cu at (33.3, 108.0)
- added MX_F4: MX-LED, MX_Only:MXOnly-1U, F.Cu at (33.3, 117.5)
- added MX_F5: MX-LED, MX_Only:MXOnly-1U, F.Cu at (347.7, 41.3)
- added MX_F6: MX-LED, MX_Only:MXOnly-1U, F.Cu at (347.7, 60.3)
- added MX_F6V1: MX-LED, MX_Only:MXOnly-2U, F.Cu at (347.7, 69.8)
- added MX_F7: MX-LED, MX_Only:MXOnly-1U, F.Cu at (347.7, 79.4)
- added MX_F8: MX-LED, MX_Only:MXOnly-1U, F.Cu at (347.7, 98.4)
- added MX_F8V1: MX-LED, MX_Only:MXOnly-2U, F.Cu at (347.7, 108.0)
- added MX_F9: MX-LED, MX_Only:MXOnly-1U, F.Cu at (347.7, 117.5)
- added MX_G1: MX-LED, MX_Only:MXOnly-1U, F.Cu at (166.7, 79.4)
- added MX_H1: MX-LED, MX_Only:MXOnly-1U, F.Cu at (185.7, 79.4)
- added MX_I1: MX-LED, MX_Only:MXOnly-1U, F.Cu at (219.1, 60.3)
- added MX_J1: MX-LED, MX_Only:MXOnly-1U, F.Cu at (204.8, 79.4)
- added MX_K1: MX-LED, MX_Only:MXOnly-1U, F.Cu at (223.8, 79.4)
- added MX_L1: MX-LED, MX_Only:MXOnly-1U, F.Cu at (242.9, 79.4)
- added MX_LALT1: MX-LED, MX_Only:MXOnly-1.5U, F.Cu at (109.5, 117.5)
- added MX_LCTRL1: MX-LED, MX_Only:MXOnly-1.5U, F.Cu at (61.9, 117.5)
- added MX_LGUI1: MX-LED, MX_Only:MXOnly-1U, F.Cu at (85.7, 117.5)
- added MX_LSHIFT1: MX-LED, MX_Only:MXOnly-2.25U, F.Cu at (69.1, 98.4)
- added MX_M1: MX-LED, MX_Only:MXOnly-1U, F.Cu at (214.3, 98.4)
- added MX_N1: MX-LED, MX_Only:MXOnly-1U, F.Cu at (195.3, 98.4)
- added MX_O1: MX-LED, MX_Only:MXOnly-1U, F.Cu at (238.1, 60.3)
- added MX_P1: MX-LED, MX_Only:MXOnly-1U, F.Cu at (257.2, 60.3)
- added MX_Q1: MX-LED, MX_Only:MXOnly-1U, F.Cu at (85.7, 60.3)
- added MX_R1: MX-LED, MX_Only:MXOnly-1U, F.Cu at (142.9, 60.3)
- added MX_RALT1: MX-LED, MX_Only:MXOnly-1.5U, F.Cu at (271.5, 117.5)
- added MX_RCTRL1: MX-LED, MX_Only:MXOnly-1.5U, F.Cu at (319.1, 117.5)
- added MX_RGUI1: MX-LED, MX_Only:MXOnly-1U, F.Cu at (295.3, 117.5)
- added MX_RSHIFT1: MX-LED, MX_Only:MXOnly-2.75U, F.Cu at (307.2, 98.4)
- added MX_RSHIFTSPLIT1: MX-LED, MX_Only:MXOnly-1.75U, F.Cu at (297.7, 98.4)
- added MX_S1: MX-LED, MX_Only:MXOnly-1U, F.Cu at (109.5, 79.4)
- added MX_SPACE1: MX-LED, MX_Only:MXOnly-7U-ReversedStabilizers, F.Cu at (190.5, 117.5)
- added MX_SPLITFN1: MX-LED, MX_Only:MXOnly-1U, F.Cu at (323.9, 98.4)
- added MX_T1: MX-LED, MX_Only:MXOnly-1U, F.Cu at (161.9, 60.3)
- added MX_TAB1: MX-LED, MX_Only:MXOnly-1.5U, F.Cu at (61.9, 60.3)
- added MX_TILDE1: MX-LED, MX_Only:MXOnly-1U, F.Cu at (57.1, 41.3)
- added MX_U1: MX-LED, MX_Only:MXOnly-1U, F.Cu at (200.0, 60.3)
- added MX_V1: MX-LED, MX_Only:MXOnly-1U, F.Cu at (157.2, 98.4)
- added MX_W1: MX-LED, MX_Only:MXOnly-1U, F.Cu at (104.8, 60.3)
- added MX_X1: MX-LED, MX_Only:MXOnly-1U, F.Cu at (119.1, 98.4)
- added MX_Y1: MX-LED, MX_Only:MXOnly-1U, F.Cu at (181.0, 60.3)
- added MX_Z1: MX-LED, MX_Only:MXOnly-1U, F.Cu at (100.0, 98.4)
- added MX_[1: MX-LED, MX_Only:MXOnly-1U, F.Cu at (276.2, 60.3)
- added MX_\1: MX-LED, MX_Only:MXOnly-1.5U, F.Cu at (319.1, 60.3)
- added MX_]1: MX-LED, MX_Only:MXOnly-1U, F.Cu at (295.3, 60.3)
- added Q1: 2N7002, Package_TO_SOT_SMD:SOT-23, B.Cu at (64.8, 107.2)
- added R10: 1k, Resistor_SMD:R_0603_1608Metric, B.Cu at (84.1, 46.8)
- added R11: 1k, Resistor_SMD:R_0603_1608Metric, B.Cu at (93.7, 65.9)
- added R12: 1k, Resistor_SMD:R_0603_1608Metric, B.Cu at (98.4, 84.9)
- added R13: 1k, Resistor_SMD:R_0603_1608Metric, B.Cu at (108.0, 104.0)
- added R14: 1k, Resistor_SMD:R_0603_1608Metric, B.Cu at (93.7, 123.0)
- added R15: 1k, Resistor_SMD:R_0603_1608Metric, B.Cu at (103.2, 46.8)
- added R16: 1k, Resistor_SMD:R_0603_1608Metric, B.Cu at (112.7, 65.9)
- added R17: 1k, Resistor_SMD:R_0603_1608Metric, B.Cu at (117.5, 84.9)
- added R18: 1k, Resistor_SMD:R_0603_1608Metric, B.Cu at (127.0, 104.0)
- added R19: 1k, Resistor_SMD:R_0603_1608Metric, B.Cu at (117.5, 123.0)
- added R20: 1k, Resistor_SMD:R_0603_1608Metric, B.Cu at (122.2, 46.8)
- added R21: 1k, Resistor_SMD:R_0603_1608Metric, B.Cu at (131.8, 65.9)
- added R22: 1k, Resistor_SMD:R_0603_1608Metric, B.Cu at (136.5, 84.9)
- added R23: 1k, Resistor_SMD:R_0603_1608Metric, B.Cu at (146.1, 104.0)
- added R24: 1k, Resistor_SMD:R_0603_1608Metric, B.Cu at (141.3, 46.8)
- added R25: 1k, Resistor_SMD:R_0603_1608Metric, B.Cu at (150.8, 65.9)
- added R26: 1k, Resistor_SMD:R_0603_1608Metric, B.Cu at (155.6, 84.9)
- added R27: 1k, Resistor_SMD:R_0603_1608Metric, B.Cu at (165.1, 104.0)
- added R28: 1k, Resistor_SMD:R_0603_1608Metric, B.Cu at (160.3, 46.8)
- added R29: 1k, Resistor_SMD:R_0603_1608Metric, B.Cu at (169.9, 65.9)
- added R30: 1k, Resistor_SMD:R_0603_1608Metric, B.Cu at (174.6, 84.9)
- added R31: 1k, Resistor_SMD:R_0603_1608Metric, B.Cu at (184.2, 104.0)
- added R32: 1k, Resistor_SMD:R_0603_1608Metric, B.Cu at (179.4, 46.8)
- added R33: 1k, Resistor_SMD:R_0603_1608Metric, B.Cu at (188.9, 65.9)
- added R34: 1k, Resistor_SMD:R_0603_1608Metric, B.Cu at (193.7, 84.9)
- added R35: 1k, Resistor_SMD:R_0603_1608Metric, B.Cu at (203.2, 104.0)
- added R36: 1k, Resistor_SMD:R_0603_1608Metric, B.Cu at (198.4, 123.0)
- added R37: 1k, Resistor_SMD:R_0603_1608Metric, B.Cu at (198.4, 46.8)
- added R38: 1k, Resistor_SMD:R_0603_1608Metric, B.Cu at (208.0, 65.9)
- added R39: 1k, Resistor_SMD:R_0603_1608Metric, B.Cu at (212.7, 84.9)
- added R40: 1k, Resistor_SMD:R_0603_1608Metric, B.Cu at (222.2, 104.0)
- added R41: 1k, Resistor_SMD:R_0603_1608Metric, B.Cu at (217.5, 46.8)
- added R42: 1k, Resistor_SMD:R_0603_1608Metric, B.Cu at (227.0, 65.9)
- added R43: 1k, Resistor_SMD:R_0603_1608Metric, B.Cu at (231.8, 84.9)
- added R44: 1k, Resistor_SMD:R_0603_1608Metric, B.Cu at (241.3, 104.0)
- added R45: 1k, Resistor_SMD:R_0603_1608Metric, B.Cu at (236.5, 46.8)
- added R46: 1k, Resistor_SMD:R_0603_1608Metric, B.Cu at (246.1, 65.9)
- added R47: 1k, Resistor_SMD:R_0603_1608Metric, B.Cu at (250.8, 84.9)
- added R48: 1k, Resistor_SMD:R_0603_1608Metric, B.Cu at (260.4, 104.0)
- added R49: 1k, Resistor_SMD:R_0603_1608Metric, B.Cu at (279.4, 123.0)
- added R5: 1k, Resistor_SMD:R_0603_1608Metric, B.Cu at (42.1, 108.7)
- added R50: 1k, Resistor_SMD:R_0603_1608Metric, B.Cu at (255.6, 46.8)
- added R51: 1k, Resistor_SMD:R_0603_1608Metric, B.Cu at (265.1, 65.9)
- added R52: 1k, Resistor_SMD:R_0603_1608Metric, B.Cu at (269.9, 84.9)
- added R53: 1k, Resistor_SMD:R_0603_1608Metric, B.Cu at (279.4, 104.0)
- added R54: 1k, Resistor_SMD:R_0603_1608Metric, B.Cu at (303.2, 123.0)
- added R55: 1k, Resistor_SMD:R_0603_1608Metric, B.Cu at (274.6, 46.8)
- added R56: 1k, Resistor_SMD:R_0603_1608Metric, B.Cu at (284.2, 65.9)
- added R57: 1k, Resistor_SMD:R_0603_1608Metric, B.Cu at (288.9, 84.9)
- added R58: 1k, Resistor_SMD:R_0603_1608Metric, B.Cu at (289.7, 104.0)
- added R59: 1k, Resistor_SMD:R_0603_1608Metric, B.Cu at (327.0, 123.0)
- added R6: 1k, Resistor_SMD:R_0603_1608Metric, B.Cu at (65.1, 46.8)
- added R60: 1k, Resistor_SMD:R_0603_1608Metric, B.Cu at (293.7, 46.8)
- added R61: 1k, Resistor_SMD:R_0603_1608Metric, B.Cu at (303.2, 65.9)
- added R62: 1k, Resistor_SMD:R_0603_1608Metric, B.Cu at (319.9, 84.9)
- added R63: 1k, Resistor_SMD:R_0603_1608Metric, B.Cu at (315.9, 104.0)
- added R64: 1k, Resistor_SMD:R_0603_1608Metric, B.Cu at (296.9, 46.8)
- added R65: 1k, Resistor_SMD:R_0603_1608Metric, B.Cu at (311.1, 65.9)
- added R66: 1k, Resistor_SMD:R_0603_1608Metric, B.Cu at (331.8, 46.8)
- added R67: 1k, Resistor_SMD:R_0603_1608Metric, B.Cu at (41.3, 46.8)
- added R68: 1k, Resistor_SMD:R_0603_1608Metric, B.Cu at (338.9, 69.1)
- added R69: 1k, Resistor_SMD:R_0603_1608Metric, B.Cu at (338.9, 70.6)
- added R7: 1k, Resistor_SMD:R_0603_1608Metric, B.Cu at (69.8, 65.9)
- added R70: 1k, Resistor_SMD:R_0603_1608Metric, B.Cu at (338.9, 107.2)
- added R71: 1k, Resistor_SMD:R_0603_1608Metric, B.Cu at (338.9, 108.7)
- added R72: 1k, Resistor_SMD:R_0603_1608Metric, B.Cu at (339.7, 46.8)
- added R8: 1k, Resistor_SMD:R_0603_1608Metric, B.Cu at (77.0, 104.0)
- added R9: 1k, Resistor_SMD:R_0603_1608Metric, B.Cu at (69.8, 123.0)
- added RC1: 22, Resistor_SMD:R_0603_1608Metric, B.Cu at (48.0, 57.1)
- added RC2: 22, Resistor_SMD:R_0603_1608Metric, B.Cu at (50.9, 58.4)
- added RC3: 1.5k, Resistor_SMD:R_0603_1608Metric, B.Cu at (64.6, 103.6)
- added RC4: 10k, Resistor_SMD:R_0603_1608Metric, B.Cu at (51.6, 108.0)
- R1, R2: value 22 -> 1k
- R3, R4: value 10k -> 1k
- moved D50 79.0 mm to (279.4, 117.5)
- moved D15 76.1 mm to (93.7, 117.5)
- moved D20 75.6 mm to (117.5, 117.5)
- moved D37 75.4 mm to (198.4, 117.5)
- moved D60 61.1 mm to (327.0, 117.5)
- moved D55 59.4 mm to (303.2, 117.5)
- moved D32 56.6 mm to (184.2, 98.4)
- moved D24 56.6 mm to (146.1, 98.4)
- moved D28 56.6 mm to (165.1, 98.4)
- moved D41 56.6 mm to (222.2, 98.4)
- moved D45 56.6 mm to (241.3, 98.4)
- moved D54 56.6 mm to (279.4, 98.4)
- moved D59 56.5 mm to (289.7, 98.4)
- moved D58 55.0 mm to (288.9, 79.4)
- moved D62 48.4 mm to (303.2, 60.3)
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Connections:
- D10 pad 1: ROW4 -> ROW9
- D12 pad 1: ROW1 -> ROW2
- D13 pad 1: ROW2 -> ROW4
- D14 pad 1: ROW3 -> ROW6
- D15 pad 1: ROW0 -> ROW8
- D17 pad 1: ROW2 -> ROW3
- D18 pad 1: ROW3 -> ROW5
- D19 pad 1: ROW4 -> ROW7
- D2 pad 1: ROW1 -> ROW2
- D20 pad 1: ROW0 -> ROW9
- D21 pad 1: ROW1 -> ROW0
- D23 pad 1: ROW3 -> ROW4
- D24 pad 1: ROW0 -> ROW6
- D26 pad 1: ROW2 -> ROW3
- D27 pad 1: ROW3 -> ROW5
- D28 pad 1: ROW0 -> ROW7
- D29 pad 1: ROW1 -> ROW0
- D3 pad 1: ROW2 -> ROW4
- D31 pad 1: ROW3 -> ROW4
- D32 pad 1: ROW0 -> ROW6
- D34 pad 1: ROW2 -> ROW3
- D35 pad 1: ROW3 -> ROW5
- D36 pad 1: ROW4 -> ROW7
- D37 pad 1: ROW0 -> ROW9
- D38 pad 1: ROW1 -> ROW0
- D4 pad 1: ROW3 -> ROW6
- D40 pad 1: ROW3 -> ROW4
- D41 pad 1: ROW0 -> ROW6
- D43 pad 1: ROW2 -> ROW3
- D44 pad 1: ROW3 -> ROW5
- D45 pad 1: ROW0 -> ROW7
- D46 pad 1: ROW1 -> ROW0
- D48 pad 1: ROW3 -> ROW4
- D49 pad 1: ROW4 -> ROW6
- D5 pad 1: ROW4 -> ROW8
- D50 pad 1: ROW0 -> ROW8
- D52 pad 1: ROW2 -> ROW3
- D53 pad 1: ROW3 -> ROW5
- D54 pad 1: ROW0 -> ROW7
- D55 pad 1: ROW1 -> ROW9
- D56 pad 1: ROW2 -> ROW0
- D57 pad 1: ROW3 -> ROW2
- D59 pad 1: ROW0 -> ROW6
- D6 pad 1: ROW0 -> ROW1
- D60 pad 1: ROW1 -> ROW8
- D61 pad 1: ROW2 -> ROW1
- D63 pad 1: ROW0 -> ROW5
- D64 pad 1: ROW1 -> ROW7
- D65 pad 1: ROW2 -> ROW0
- D66 pad 1: ROW0 -> ROW2
- D67 pad 1: ROW1 -> ROW4
- D68 pad 1: ROW2 -> ROW1
- D7 pad 1: ROW1 -> ROW3
- D70 pad 1: ROW4 -> ROW5
- D8 pad 1: ROW2 -> ROW5
- D9 pad 1: ROW3 -> ROW7
- R1 pad 1: Net-(R1-Pad1) -> CAPS_LEDGND
- R1 pad 2: D- -> Net-(JP3-Pad2)
- R2 pad 1: Net-(R2-Pad1) -> Net-(MX_F1-Pad4)
- R2 pad 2: D+ -> LEDGND
- R3 pad 1: +5V -> Net-(MX_F2-Pad4)
- R3 pad 2: Net-(R3-Pad2) -> LEDGND
- R4 pad 1: Net-(R4-Pad1) -> Net-(MX_F3-Pad4)
- R4 pad 2: GND -> LEDGND
- U2 pad 10: ROW2 -> TGR_IND
- U2 pad 11: ROW1 -> CAPS_IND
- U2 pad 13: Net-(R3-Pad2) -> RESET
- U2 pad 18: ROW0 -> ROW9
- U2 pad 19: COL4 -> ROW8
- U2 pad 20: COL3 -> ROW7
- U2 pad 21: COL2 -> ROW6
- U2 pad 22: COL1 -> Net-(U2-Pad22)
- U2 pad 25: COL5 -> Net-(RC3-Pad2)
- U2 pad 26: COL6 -> ROW4
- U2 pad 27: COL7 -> ROW5
- U2 pad 28: COL8 -> ROW3
- U2 pad 29: COL9 -> ROW2
- U2 pad 3: Net-(R1-Pad1) -> Net-(RC1-Pad1)
- U2 pad 30: COL10 -> ROW1
- U2 pad 31: COL11 -> ROW0
- U2 pad 32: COL12 -> COL6
- U2 pad 33: Net-(R4-Pad1) -> Net-(RC4-Pad1)
- U2 pad 36: COL14 -> COL5
- U2 pad 37: COL13 -> COL4
- U2 pad 38: COL15 -> COL3
- U2 pad 39: COL0 -> COL2
- U2 pad 4: Net-(R2-Pad1) -> Net-(RC2-Pad1)
- U2 pad 40: ROW4 -> COL1
- U2 pad 41: ROW3 -> COL0
- U2 pad 8: Net-(U2-Pad8) -> COL7
- U2 pad 9: Net-(U2-Pad9) -> ESC_IND
Routing:
- net +5V: track 67.4 -> 1136.4 mm, vias 7 -> 0
- net LEDGND: track 0.00 -> 887.0 mm
- net COL14: track 407.3 -> 0.00 mm, vias 1 -> 0
- net COL15: track 406.4 -> 0.00 mm
- net COL13: track 382.0 -> 0.00 mm, vias 1 -> 0
- net COL12: track 357.3 -> 0.00 mm, vias 1 -> 0
- net COL11: track 327.2 -> 0.00 mm, vias 1 -> 0
- net COL10: track 305.1 -> 0.00 mm, vias 1 -> 0
- net ROW5: track 0.00 -> 278.3 mm
- net COL9: track 259.7 -> 0.00 mm, vias 1 -> 0
- net ROW7: track 0.00 -> 246.5 mm
- net ROW9: track 0.00 -> 238.1 mm
- net COL8: track 234.2 -> 0.00 mm, vias 1 -> 0
- net ROW8: track 0.00 -> 215.6 mm
- net COL6: track 194.1 -> 0.00 mm, vias 1 -> 0
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- removed copper zone on B.Cu, net GND
Other:
- outline, holes or cut-outs redrawn
- net class Power: trace_width 0.254 -> 0.381
