File: _autosave-rei_pcb.sch (KiCad schematic (older format))
At the start: 243 parts, among them J1 SM04B-SRSS-TB(LF)(SN), J2 AVR-ISP-6, Q1 Q_NPN_BCE, U2 ATmega32U4RC-MU, Y1 16MHz

Commit message: Updating pcb
Parts:
- removed Q1: Q_NPN_BCE, Package_TO_SOT_SMD:SOT-223-3_TabPin2, symbol Device:Q_NPN_BCE
- added Q1: 2N7002, Package_TO_SOT_SMD:SOT-23, symbol Transistor_FET:2N7002
- MX_CLOCKSTEP1: footprint MX_Only:MXOnly-1.25U -> MX_Only:MXOnly-1.25U-FLIPPED
Connections:
- wire segments 759 -> 761
Other:
- moved on the sheet: RC3
Changed lines of the file:
@@
 F 0 "MX_CLOCKSTEP1" H 5682 11524 60  0000 C CNN
 F 1 "MX-LED" H 5682 11450 20  0000 C CNN
-F 2 "MX_Only:MXOnly-1.25U" H 4975 11275 60  0001 C CNN
+F 2 "MX_Only:MXOnly-1.25U-FLIPPED" H 4975 11275 60  0001 C CNN
 F 3 "" H 4975 11275 60  0001 C CNN
 	1    5600 11300
@@
 Wire Wire Line
 	14050 10800 14050 11000
-Wire Wire Line
-	14050 11000 13450 11000
 Connection ~ 13450 11000
 Wire Wire Line
@@
 Text GLabel 6600 2550 2    50   Input ~ 0
 ROW3
+Text GLabel 6600 3950 2    50   Input ~ 0
+ROW4
 Text GLabel 6600 4050 2    50   Input ~ 0
-ROW4
-Text GLabel 6600 3950 2    50   Input ~ 0
 ROW5
-Text GLabel 6600 3850 2    50   Input ~ 0
+Text GLabel 6600 3650 2    50   Input ~ 0
 ROW6
-Text GLabel 6600 3750 2    50   Input ~ 0
+Text GLabel 6600 3550 2    50   Input ~ 0
 ROW7
-Text GLabel 6600 3650 2    50   Input ~ 0
+Text GLabel 6600 3450 2    50   Input ~ 0
 ROW8
-Text GLabel 6600 3550 2    50   Input ~ 0
+Text GLabel 6600 3350 2    50   Input ~ 0
 ROW9
 Text GLabel 5400 2150 0    50   Input ~ 0
@@
 TGR_IND
 Wire Wire Line
-	6600 2850 7400 2850
+	6600 3750 7400 3750
 $Comp
 L Device:R_Small RC3
 U 1 1 66741666
-P 7500 2850
-F 0 "RC3" V 7304 2850 50  0000 C CNN
-F 1 "1.5k" V 7395 2850 50  0000 C CNN
-F 2 "Resistor_SMD:R_0603_1608Metric" H 7500 2850 50  0001 C CNN
-F 3 "~" H 7500 2850 50  0001 C CNN
-	1    7500 2850
+P 7500 3750
+F 0 "RC3" V 7304 3750 50  0000 C CNN
+F 1 "1.5k" V 7395 3750 50  0000 C CNN
+F 2 "Resistor_SMD:R_0603_1608Metric" H 7500 3750 50  0001 C CNN
+F 3 "~" H 7500 3750 50  0001 C CNN
+	1    7500 3750
 	0    1    1    0
 $EndComp
 Wire Wire Line
-	7600 2850 8100 2850
-$Comp
-L Device:Q_NPN_BCE Q1
-U 1 1 667D88BC
-P 8300 2850
-F 0 "Q1" H 8491 2896 50  0000 L CNN
-F 1 "Q_NPN_BCE" H 8491 2805 50  0000 L CNN
-F 2 "Package_TO_SOT_SMD:SOT-223-3_TabPin2" H 8500 2950 50  0001 C CNN
-F 3 "~" H 8300 2850 50  0001 C CNN
-	1    8300 2850
-	1    0    0    -1
-$EndComp
-Text GLabel 8400 2650 1    50   Input ~ 0
+	7600 3750 8100 3750
+Text GLabel 8400 3550 1    50   Input ~ 0
 LEDGND
 $Comp
 L power:GND #PWR015
 U 1 1 6686B41D
-P 8400 3050
-F 0 "#PWR015" H 8400 2800 50  0001 C CNN
-F 1 "GND" H 8405 2877 50  0000 C CNN
-F 2 "" H 8400 3050 50  0001 C CNN
-F 3 "" H 8400 3050 50  0001 C CNN
-	1    8400 3050
+P 8400 3950
+F 0 "#PWR015" H 8400 3700 50  0001 C CNN
+F 1 "GND" H 8405 3777 50  0000 C CNN
+F 2 "" H 8400 3950 50  0001 C CNN
+F 3 "" H 8400 3950 50  0001 C CNN
+	1    8400 3950
 	1    0    0    -1
 $EndComp
@@
 	0    -1   -1   0
 $EndComp
+Wire Wire Line
+	15250 10800 15250 11000
+Wire Wire Line
+	13450 11000 14050 11000
+Connection ~ 14050 11000
+Wire Wire Line
+	14050 11000 15250 11000
+$Comp
+L Transistor_FET:2N7002 Q1
+U 1 1 60A4084D
+P 8300 3750
+F 0 "Q1" H 8504 3796 50  0000 L CNN
+F 1 "2N7002" H 8504 3705 50  0000 L CNN
+F 2 "Package_TO_SOT_SMD:SOT-23" H 8500 3675 50  0001 L CIN
+F 3 "https://www.fairchildsemi.com/datasheets/2N/2N7002.pdf" H 8300 3750 50  0001 L CNN
+	1    8300 3750
+	1    0    0    -1
+$EndComp
 $EndSCHEMATC
